File: Mlrs_lorae5mini/mlrs_lora_e5mini.brd (EAGLE design)
At the start: 15 x 28.4 mm, 19 parts, among them U1 LoRa-E5-HF, U2 AP2112K-3.3TRG1, X1 1296-T18

Commit message: Add files via upload
Parts:
- added BOOT: (no value), jumper:SJ
- added R12: 470R, Discrete-new:R0402
- moved R1 13.5 mm to (14.0, 22.9), turned to 90 degrees
- moved D1 13.2 mm to (13.9, 19.8), turned to 270 degrees
- moved D6 13.0 mm to (1.02, 22.4)
- moved R13 13.0 mm to (1.02, 19.6)
Connections:
- new net N$1: D1.-, R1.1
- new net N$29: BOOT.2, R12.1
- net GND: now also R12.2
- net PB13/BOOT/SCK: now also BOOT.1
- net PB15/SCL: no longer D1.-, R1.1
Routing:
- net PB15/SCL: track 21.1 -> 0.00 mm
- net 3V3: track 34.6 -> 22.7 mm, vias 2 -> 0
- net PB5/LED: track 14.1 -> 21.0 mm, vias 0 -> 2
- net PA15/SDA: track 21.4 -> 15.5 mm, vias 2 -> 0
- net PB13/BOOT/SCK: track 0.00 -> 4.45 mm, vias 0 -> 1
- net TX1: track 16.5 -> 13.5 mm
- net A3: track 9.24 -> 6.29 mm
- net RX1: track 18.0 -> 15.2 mm
- net TX0: track 13.1 -> 10.6 mm
- net GND: track 10.0 -> 7.85 mm, vias 5 -> 27
- net N$29: track 0.00 -> 2.08 mm
- net N$1: track 0.00 -> 1.93 mm
- net RX0: track 10.7 -> 8.91 mm
- net RX2: track 18.3 -> 16.9 mm
- net 5V: track 19.6 -> 20.4 mm
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Other:
- board text added: "ULTRA DRONES"
