File: Mlrs_lorae5mini/mlrs_lora_e5mini.sch (EAGLE design)
At the start: 19 parts, among them U1 LoRa-E5-HF, U2 AP2112K-3.3TRG1, X1 1296-T18

Commit message: Add files via upload
Parts:
- added BOOT: (no value), jumper:SJ
- added R12: 470R, Discrete-new:RES-0402
Connections:
- new net N$1: D1.-, R1.1
- new net N$29: BOOT.2, R12.1
- net GND: now also R12.2
- net PB13/BOOT/SCK: now also BOOT.1
- net PB15/SCL: no longer D1.-, R1.1
Changed lines of the file:
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@@
 <setting verticaltext="up"/>
 </settings>
-<grid distance="0.05" unitdist="inch" unit="inch" style="lines" multiple="1" display="no" altdistance="0.01" altunitdist="inch" altunit="inch"/>
+<grid distance="0.1" unitdist="inch" unit="inch" style="lines" multiple="1" display="no" altdistance="0.01" altunitdist="inch" altunit="inch"/>
 <layers>
 <layer number="1" name="Top" color="4" fill="1" visible="no" active="no"/>
@@
 <part name="D6" library="Discrete-new" deviceset="LED" device="'0603'" value="RED"/>
 <part name="R13" library="Discrete-new" deviceset="RES" device="-0402" value="1k"/>
+<part name="BOOT" library="jumper" library_urn="urn:adsk.eagle:library:252" deviceset="SJ" device="" package3d_urn="urn:adsk.eagle:package:15471/1"/>
+<part name="G12" library="Power or GND " deviceset="GND_POWER" device=""/>
+<part name="G9" library="Power or GND " deviceset="GND_POWER" device=""/>
+<part name="R12" library="Discrete-new" deviceset="RES" device="-0402" value="470R"/>
 </parts>
 <sheets>
@@
 <attribute name="NAME" x="59.69" y="-5.08" size="1.27" layer="95" ratio="10" rot="R180"/>
 <attribute name="VALUE" x="54.61" y="-5.08" size="1.27" layer="96" ratio="10" rot="R180"/>
+</instance>
+<instance part="BOOT" gate="1" x="111.76" y="104.14" smashed="yes">
+<attribute name="NAME" x="109.22" y="106.68" size="1.778" layer="95"/>
+<attribute name="VALUE" x="109.22" y="100.33" size="1.778" layer="96"/>
+</instance>
+<instance part="G12" gate="G$1" x="124.46" y="114.3" smashed="yes" rot="R90"/>
+<instance part="G9" gate="G$1" x="132.08" y="104.14" smashed="yes" rot="R90"/>
+<instance part="R12" gate="R" x="125.73" y="104.14" smashed="yes">
+<attribute name="NAME" x="123.19" y="105.41" size="1.27" layer="95" ratio="10"/>
+<attribute name="VALUE" x="128.27" y="105.41" size="1.27" layer="96" ratio="10"/>
 </instance>
 </instances>
@@
 <label x="87.63" y="3.81" size="1.778" layer="95"/>
 </segment>
+<segment>
+<pinref part="G12" gate="G$1" pin="GND"/>
+<wire x1="115.57" y1="114.3" x2="121.412" y2="114.3" width="0.1524" layer="91"/>
+<wire x1="121.412" y1="114.3" x2="124.46" y2="114.3" width="0.1524" layer="91"/>
+<wire x1="121.412" y1="114.3" x2="121.412" y2="115.57" width="0.1524" layer="91"/>
+<junction x="121.412" y="114.3"/>
+<wire x1="121.412" y1="115.57" x2="115.57" y2="115.57" width="0.1524" layer="91"/>
+</segment>
+<segment>
+<pinref part="G9" gate="G$1" pin="GND"/>
+<wire x1="129.54" y1="104.14" x2="132.08" y2="104.14" width="0.1524" layer="91"/>
+<pinref part="R12" gate="R" pin="2"/>
+</segment>
 </net>
 <net name="PA13/SWDIO" class="0">
@@
 <label x="25.4" y="44.45" size="0.889" layer="95" ratio="12" rot="R180" xref="yes"/>
 </segment>
-<segment>
-<pinref part="D1" gate="LED" pin="-"/>
-<wire x1="77.47" y1="3.81" x2="62.23" y2="3.81" width="0.1524" layer="91"/>
-<label x="64.77" y="3.81" size="1.778" layer="95"/>
-<pinref part="R1" gate="R" pin="1"/>
-</segment>
 </net>
 <net name="RST" class="0">
@@
 <label x="80.01" y="44.45" size="0.889" layer="95" ratio="12" xref="yes"/>
 </segment>
+<segment>
+<wire x1="104.14" y1="115.57" x2="104.14" y2="114.3" width="0.1524" layer="91"/>
+<wire x1="107.95" y1="114.3" x2="104.14" y2="114.3" width="0.1524" layer="91"/>
+<wire x1="107.95" y1="115.57" x2="104.14" y2="115.57" width="0.1524" layer="91"/>
+<wire x1="104.14" y1="115.57" x2="99.06" y2="115.57" width="0.1524" layer="91"/>
+<junction x="104.14" y="115.57"/>
+<label x="99.06" y="115.57" size="0.889" layer="95" ratio="12" rot="R180" xref="yes"/>
+</segment>
 </net>
 <net name="PA10/MOSI" class="0">
@@
 <wire x1="58.42" y1="67.31" x2="58.42" y2="74.93" width="0.1524" layer="91"/>
 <label x="58.42" y="74.93" size="0.889" layer="95" ratio="12" rot="R90" xref="yes"/>
+</segment>
+<segment>
+<label x="99.06" y="105.41" size="0.889" layer="95" ratio="12" rot="R180" xref="yes"/>
+<wire x1="102.87" y1="105.41" x2="99.06" y2="105.41" width="0.1524" layer="91"/>
+<wire x1="107.95" y1="104.14" x2="106.68" y2="104.14" width="0.1524" layer="91"/>
+<wire x1="106.68" y1="104.14" x2="102.87" y2="104.14" width="0.1524" layer="91"/>
+<wire x1="102.87" y1="104.14" x2="102.87" y2="105.41" width="0.1524" layer="91"/>
+<pinref part="BOOT" gate="1" pin="1"/>
 </segment>
 </net>
@@
 </segment>
 </net>
+<net name="N$1" class="0">
+<segment>
+<pinref part="D1" gate="LED" pin="-"/>
+<pinref part="R1" gate="R" pin="1"/>
+<wire x1="62.23" y1="3.81" x2="77.47" y2="3.81" width="0.1524" layer="91"/>
+</segment>
+</net>
+<net name="N$29" class="0">
+<segment>
+<wire x1="115.57" y1="104.14" x2="116.84" y2="104.14" width="0.1524" layer="91"/>
+<wire x1="116.84" y1="104.14" x2="121.92" y2="104.14" width="0.1524" layer="91"/>
+<pinref part="R12" gate="R" pin="1"/>
+<pinref part="BOOT" gate="1" pin="2"/>
+</segment>
+</net>
